File: synthia/synthia.kicad_sch (KiCad schematic)
At the start: 0 parts

Commit message: L
Parts:
- added U1: 74AHC04, symbol 74xx:74AHC04
Changed lines of the file:
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@@
+		)
+	)
+	(symbol
+		(lib_id "74xx:74AHC04")
+		(at 182.88 121.92 0)
+		(unit 2)
+		(exclude_from_sim no)
+		(in_bom yes)
+		(on_board yes)
+		(dnp no)
+		(fields_autoplaced yes)
+		(property "Reference" "U1"
+			(at 182.88 113.03 0)
+			(effects
+				(font
+					(size 1.27 1.27)
+				)
+			)
+		)
+		(property "Value" "74AHC04"
+			(at 182.88 115.57 0)
+			(effects
+				(font
+					(size 1.27 1.27)
+				)
+			)
+		)
+		(property "Footprint" ""
+			(at 182.88 121.92 0)
+			(effects
+				(font
+					(size 1.27 1.27)
+				)
+				(hide yes)
+			)
+		)
+		(property "Datasheet" "https://assets.nexperia.com/documents/data-sheet/74AHC_AHCT04.pdf"
+			(at 182.88 121.92 0)
+			(effects
+				(font
+					(size 1.27 1.27)
+				)
+				(hide yes)
+			)
+		)
+		(property "Description" "Hex Inverter"
+			(at 182.88 121.92 0)
+			(effects
+				(font
+					(size 1.27 1.27)
+				)
+				(hide yes)
+			)
+		)
+		(pin "13"
+		)
+		(pin "12"
+		)
+		(pin "7"
+		)
+		(pin "3"
+		)
+		(pin "10"
+		)
+		(pin "14"
+		)
+		(pin "1"
+		)
+		(pin "11"
+		)
+		(pin "2"
+		)
+		(pin "4"
+		)
+		(pin "5"
+		)
+		(pin "6"
+		)
+		(pin "9"
+		)
+		(pin "8"
+		)
+		(instances
+			(project ""
+				(path "/b7ca07b0-c23c-4333-a610-582d2798793b"
+					(reference "U1")
+					(unit 2)
+				)
+			)
+		)
+	)
+	(symbol
+		(lib_id "74xx:74AHC04")
+		(at 134.62 137.16 0)
+		(unit 1)
+		(exclude_from_sim no)
+		(in_bom yes)
+		(on_board yes)
+		(dnp no)
+		(fields_autoplaced yes)
+		(property "Reference" "U1"
+			(at 134.62 128.27 0)
+			(effects
+				(font
+					(size 1.27 1.27)
+				)
+			)
+		)
+		(property "Value" "74AHC04"
+			(at 134.62 130.81 0)
+			(effects
+				(font
+					(size 1.27 1.27)
+				)
+			)
+		)
+		(property "Footprint" ""
+			(at 134.62 137.16 0)
+			(effects
+				(font
+					(size 1.27 1.27)
+				)
+				(hide yes)
+			)
+		)
+		(property "Datasheet" "https://assets.nexperia.com/documents/data-sheet/74AHC_AHCT04.pdf"
+			(at 134.62 137.16 0)
+			(effects
+				(font
+					(size 1.27 1.27)
+				)
+				(hide yes)
+			)
+		)
+		(property "Description" "Hex Inverter"
+			(at 134.62 137.16 0)
+			(effects
+				(font
+					(size 1.27 1.27)
+				)
+				(hide yes)
+			)
+		)
+		(pin "13"
+		)
+		(pin "12"
+		)
+		(pin "7"
+		)
+		(pin "3"
+		)
+		(pin "10"
+		)
+		(pin "14"
+		)
+		(pin "1"
+		)
+		(pin "11"
+		)
+		(pin "2"
+		)
+		(pin "4"
+		)
+		(pin "5"
+		)
+		(pin "6"
+		)
+		(pin "9"
+		)
+		(pin "8"
+		)
+		(instances
+			(project ""
+				(path "/b7ca07b0-c23c-4333-a610-582d2798793b"
+					(reference "U1")
+					(unit 1)
+				)
+			)
 		)
 	)

Commit message: Meaningful Commit Message (Test)
Parts:
- removed U1: 74AHC04, symbol 74xx:74AHC04
Changed lines of the file:
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@@
-		)
-	)
-	(symbol
-		(lib_id "74xx:74AHC04")
-		(at 182.88 121.92 0)
-		(unit 2)
-		(exclude_from_sim no)
-		(in_bom yes)
-		(on_board yes)
-		(dnp no)
-		(fields_autoplaced yes)
-		(property "Reference" "U1"
-			(at 182.88 113.03 0)
-			(effects
-				(font
-					(size 1.27 1.27)
-				)
-			)
-		)
-		(property "Value" "74AHC04"
-			(at 182.88 115.57 0)
-			(effects
-				(font
-					(size 1.27 1.27)
-				)
-			)
-		)
-		(property "Footprint" ""
-			(at 182.88 121.92 0)
-			(effects
-				(font
-					(size 1.27 1.27)
-				)
-				(hide yes)
-			)
-		)
-		(property "Datasheet" "https://assets.nexperia.com/documents/data-sheet/74AHC_AHCT04.pdf"
-			(at 182.88 121.92 0)
-			(effects
-				(font
-					(size 1.27 1.27)
-				)
-				(hide yes)
-			)
-		)
-		(property "Description" "Hex Inverter"
-			(at 182.88 121.92 0)
-			(effects
-				(font
-					(size 1.27 1.27)
-				)
-				(hide yes)
-			)
-		)
-		(pin "13"
-		)
-		(pin "12"
-		)
-		(pin "7"
-		)
-		(pin "3"
-		)
-		(pin "10"
-		)
-		(pin "14"
-		)
-		(pin "1"
-		)
-		(pin "11"
-		)
-		(pin "2"
-		)
-		(pin "4"
-		)
-		(pin "5"
-		)
-		(pin "6"
-		)
-		(pin "9"
-		)
-		(pin "8"
-		)
-		(instances
-			(project ""
-				(path "/b7ca07b0-c23c-4333-a610-582d2798793b"
-					(reference "U1")
-					(unit 2)
-				)
-			)
-		)
-	)
-	(symbol
-		(lib_id "74xx:74AHC04")
-		(at 134.62 137.16 0)
-		(unit 1)
-		(exclude_from_sim no)
-		(in_bom yes)
-		(on_board yes)
-		(dnp no)
-		(fields_autoplaced yes)
-		(property "Reference" "U1"
-			(at 134.62 128.27 0)
-			(effects
-				(font
-					(size 1.27 1.27)
-				)
-			)
-		)
-		(property "Value" "74AHC04"
-			(at 134.62 130.81 0)
-			(effects
-				(font
-					(size 1.27 1.27)
-				)
-			)
-		)
-		(property "Footprint" ""
-			(at 134.62 137.16 0)
-			(effects
-				(font
-					(size 1.27 1.27)
-				)
-				(hide yes)
-			)
-		)
-		(property "Datasheet" "https://assets.nexperia.com/documents/data-sheet/74AHC_AHCT04.pdf"
-			(at 134.62 137.16 0)
-			(effects
-				(font
-					(size 1.27 1.27)
-				)
-				(hide yes)
-			)
-		)
-		(property "Description" "Hex Inverter"
-			(at 134.62 137.16 0)
-			(effects
-				(font
-					(size 1.27 1.27)
-				)
-				(hide yes)
-			)
-		)
-		(pin "13"
-		)
-		(pin "12"
-		)
-		(pin "7"
-		)
-		(pin "3"
-		)
-		(pin "10"
-		)
-		(pin "14"
-		)
-		(pin "1"
-		)
-		(pin "11"
-		)
-		(pin "2"
-		)
-		(pin "4"
-		)
-		(pin "5"
-		)
-		(pin "6"
-		)
-		(pin "9"
-		)
-		(pin "8"
-		)
-		(instances
-			(project ""
-				(path "/b7ca07b0-c23c-4333-a610-582d2798793b"
-					(reference "U1")
-					(unit 1)
-				)
-			)
 		)
 	)

Commit message: This has the power part made out k
Parts:
- added BT1: 9V, symbol Device:Battery
- added C1: 330nF, symbol Device:C_Small
- added C2: 100nF, symbol Device:C_Small
- added D1: 1N4742A, Diode_THT:D_DO-41_SOD81_P10.16mm_Horizontal, symbol Diode:1N47xxA
- added Q1: IRF9540N, Package_TO_SOT_THT:TO-220-3_Vertical, symbol Transistor_FET:IRF9540N
- added R2: 10k, symbol Device:R_US
- added U1: L78M05CV, Package_TO_SOT_THT:TO-220-3_Vertical, symbol Regulator_Linear:LD1117V
Connections:
- net +5V: now also C2.1, U1.2 (VO)
- new net: C1.1, D1.1 (K), Q1.3 (S), U1.3 (VI)
- new net: D1.2 (A), Q1.1 (G), R2.1
- new net +9V: BT1.1 (+), Q1.2 (D)
- new net GND: BT1.2 (-), C1.2, C2.2, R2.2, U1.1 (GND)

Commit message: Stuff from this meeting
Parts:
- added D10, D11, D12, D13, D14, D15, D16, D17, D18, D19, D2, D20, D21, D22, D23, D24, D25, D26, D27, D28, D29, D3, D30, D31, D32, D33, D34, D35, D36, D37, D4, D5, D6, D7, D8, D9: 1N4001, Diode_THT:D_DO-41_SOD81_P10.16mm_Horizontal, symbol Diode:1N4001
- added R10, R11, R12, R13, R14, R15, R16, R17, R18, R19, R20, R21, R22, R23, R24, R25, R26, R27, R28, R29, R3, R30, R31, R32, R33, R34, R35, R36, R37, R38, R39, R4, R5, R6, R7, R8, R9: 100k, symbol Device:R_US
- added SW1, SW10, SW11, SW12, SW13, SW14, SW15, SW16, SW17, SW18, SW19, SW2, SW20, SW21, SW22, SW23, SW24, SW25, SW26, SW27, SW28, SW29, SW3, SW30, SW31, SW32, SW33, SW34, SW35, SW36, SW4, SW5, SW6, SW7, SW8, SW9: SW_SPST, symbol Switch:SW_SPST
Connections:
- net GND: now also R10.2, R11.2, R12.2, R13.2, R14.2, R3.2, R39.1, R4.2, R5.2, R6.2, R7.2, R8.2, R9.2
- new net: D11.2 (A), SW10.2 (B)
- new net: R15.2, R16.1
- new net: D14.2 (A), SW13.2 (B)
- new net: D8.2 (A), SW7.2 (B)
- new net: R32.2, R35.1, R36.2
- new net: R26.1, R31.2, R35.2
- new net: D35.2 (A), SW34.2 (B)
- new net: R38.1, R39.2
- new net: R34.2, R37.1, R38.2
- new net: D31.2 (A), SW30.2 (B)
- new net: R18.1, R19.2, R20.2
- new net: D36.2 (A), SW35.2 (B)
- new net: R17.2, R19.1
- new net: D22.2 (A), SW21.2 (B)
- new net: D33.2 (A), SW32.2 (B)
- new net: D13.2 (A), SW12.2 (B)
- new net: D19.2 (A), SW18.2 (B)
- new net: D6.2 (A), SW5.2 (B)
- new net: D2.2 (A), SW1.2 (B)
- new net: D30.2 (A), SW29.2 (B)
- new net: D18.2 (A), SW17.2 (B)
- new net: D29.2 (A), SW28.2 (B)
- new net: D21.2 (A), SW20.2 (B)
- new net: R30.2, R34.1
- new net: D27.2 (A), SW26.2 (B)
- new net: D9.2 (A), SW8.2 (B)
- new net: D3.2 (A), SW2.2 (B)
- new net: D10.2 (A), SW9.2 (B)
- new net: D20.2 (A), SW19.2 (B)
- new net: D5.2 (A), SW4.2 (B)
- new net: D7.2 (A), SW6.2 (B)
- new net: R29.2, R33.1
- new net: R33.2, R36.1, R37.2
- new net: R21.2, R23.1
- new net: R22.2, R24.1
- new net: D28.2 (A), SW27.2 (B)
- new net: D4.2 (A), SW3.2 (B)
- new net: D17.2 (A), SW16.2 (B)
- new net: D37.2 (A), SW36.2 (B)
- new net: R27.2, R31.1
- new net: R24.2, R25.1, R26.2
- new net: D32.2 (A), SW31.2 (B)
- new net: D24.2 (A), SW23.2 (B)
- new net: D26.2 (A), SW25.2 (B)
- new net: D34.2 (A), SW33.2 (B)
- new net: R20.1, R23.2, R25.2
- new net: D25.2 (A), SW24.2 (B)
- new net: D12.2 (A), SW11.2 (B)
- new net: D15.2 (A), SW14.2 (B)
- new net: R28.2, R32.1
- new net: D23.2 (A), SW22.2 (B)
- new net: D16.2 (A), SW15.2 (B)
- new net DACin0: R30.1
- new net DACin1: R29.1
- new net DACin2: R28.1
- new net DACin3: R27.1
- new net DACin4: R22.1
- new net DACin5: R21.1
- new net DACin6: R17.1
- new net DACin7: R15.1
- new net DACout: R16.2, R18.2
- new net ScanCol0: SW1.1 (A), SW13.1 (A), SW14.1 (A), SW15.1 (A), SW16.1 (A), SW25.1 (A), SW26.1 (A), SW27.1 (A), SW28.1 (A), SW4.1 (A), SW7.1 (A), SW8.1 (A)
- new net ScanCol1: SW10.1 (A), SW17.1 (A), SW18.1 (A), SW19.1 (A), SW2.1 (A), SW20.1 (A), SW29.1 (A), SW30.1 (A), SW31.1 (A), SW32.1 (A), SW5.1 (A), SW9.1 (A)
- new net ScanCol2: SW11.1 (A), SW12.1 (A), SW21.1 (A), SW22.1 (A), SW23.1 (A), SW24.1 (A), SW3.1 (A), SW33.1 (A), SW34.1 (A), SW35.1 (A), SW36.1 (A), SW6.1 (A)
- new net ScanRow0: D2.1 (K), D3.1 (K), D4.1 (K), R3.1
- new net ScanRow1: D5.1 (K), D6.1 (K), D7.1 (K), R4.1
- new net ScanRow10: D28.1 (K), D32.1 (K), D36.1 (K), R13.1
- new net ScanRow11: D29.1 (K), D33.1 (K), D37.1 (K), R14.1
- new net ScanRow2: D10.1 (K), D12.1 (K), D8.1 (K), R5.1
- new net ScanRow3: D11.1 (K), D13.1 (K), D9.1 (K), R6.1
- new net ScanRow4: D14.1 (K), D18.1 (K), D22.1 (K), R7.1
- new net ScanRow5: D15.1 (K), D19.1 (K), D23.1 (K), R8.1
- new net ScanRow6: D16.1 (K), D20.1 (K), D24.1 (K), R9.1
- new net ScanRow7: D17.1 (K), D21.1 (K), D25.1 (K), R10.1
- new net ScanRow8: D26.1 (K), D30.1 (K), D34.1 (K), R11.1
- new net ScanRow9: D27.1 (K), D31.1 (K), D35.1 (K), R12.1

Commit message: updated with new symbols
Parts:
- removed D37: 1N4001, Diode_THT:D_DO-41_SOD81_P10.16mm_Horizontal, symbol Diode:1N4001
- removed R12: 100k, symbol Device:R_US
- removed SW1, SW10, SW11, SW12, SW13, SW14, SW15, SW16, SW17, SW18, SW19, SW2, SW20, SW21, SW22, SW23, SW24, SW25, SW26, SW27, SW28, SW29, SW3, SW30, SW31, SW32, SW33, SW34, SW35, SW36, SW4, SW5, SW6, SW7, SW8, SW9: SW_SPST, symbol Switch:SW_SPST
- removed U1: L78M05CV, Package_TO_SOT_THT:TO-220-3_Vertical, symbol Regulator_Linear:LD1117V
- added D38: 1N4001, Diode_THT:D_DO-41_SOD81_P10.16mm_Horizontal, symbol Diode:1N4001
- added Q2: L78M05CV, L78M05CV:TO254P450X1020X1935-3P, symbol Synthia_Symbol_Library:L78M05CV
- added R40: 100k, symbol Device:R_US
- added S1, S10, S11, S12, S13, S14, S15, S16, S17, S18, S19, S2, S20, S21, S22, S23, S24, S25, S26, S27, S28, S29, S3, S30, S31, S32, S33, S34, S35, S36, S4, S5, S6, S7, S8, S9: TL1105BF160Q, TL1105BF160Q:SW_TL1105BF160Q, symbol Synthia_Button_Symbol:TL1105BF160Q
Connections:
- net +5V: now also Q2.3 (OUT)
- net GND: now also Q2.2 (GND), R40.2
- net ScanCol0: now also S1.2, S12.2, S19.2, S20.2, S21.2, S28.2, S29.2, S30.2, S4.2, S5.2, S7.2, S9.2
- net ScanCol1: now also S11.2, S13.2, S14.2, S15.2, S2.2, S22.2, S23.2, S24.2, S31.2, S32.2, S33.2, S8.2
- net ScanCol2: now also S10.2, S16.2, S17.2, S18.2, S25.2, S26.2, S27.2, S3.2, S34.2, S35.2, S36.2, S6.2
- net ScanRow0: now also D28.1 (K), D31.1 (K), D34.1 (K), R9.1; no longer D2.1 (K), D3.1 (K), D4.1 (K), R3.1
- net ScanRow1: now also D29.1 (K), D32.1 (K), D35.1 (K), R10.1; no longer D5.1 (K), D6.1 (K), D7.1 (K), R4.1
- net ScanRow10: now also D4.1 (K), D5.1 (K), D6.1 (K); no longer D28.1 (K), D32.1 (K), D36.1 (K)
- net ScanRow11: now also D2.1 (K), D3.1 (K), D38.1 (K); no longer D29.1 (K), D33.1 (K)
- net ScanRow2: now also D30.1 (K), D33.1 (K), D36.1 (K), R11.1; no longer D10.1 (K), D12.1 (K), D8.1 (K), R5.1
- net ScanRow3: now also D19.1 (K), D22.1 (K), D25.1 (K); no longer D11.1 (K), D13.1 (K), D9.1 (K)
- net ScanRow4: now also D20.1 (K), D23.1 (K), D26.1 (K); no longer D14.1 (K), D18.1 (K), D22.1 (K)
- net ScanRow5: now also D21.1 (K), D24.1 (K), D27.1 (K); no longer D15.1 (K), D19.1 (K), D23.1 (K)
- net ScanRow6: now also D13.1 (K), D7.1 (K), R3.1; no longer D20.1 (K), D24.1 (K), R9.1
- net ScanRow7: now also D14.1 (K), D9.1 (K), R4.1; no longer D21.1 (K), D25.1 (K), R10.1
- net ScanRow8: now also D11.1 (K), D15.1 (K), D18.1 (K), R5.1; no longer D26.1 (K), D30.1 (K), D34.1 (K), R11.1
- net ScanRow9: now also D10.1 (K), D12.1 (K), D8.1 (K), R40.1; no longer D27.1 (K), D31.1 (K), D35.1 (K)
- net at D11.2 (A): now also S12.4
- net at D14.2 (A): now also S14.4
- net at D8.2 (A): now also S7.4
- net at D35.2 (A): now also S35.4
- net at C1.1, D1.1 (K), Q1.3 (S): now also Q2.1 (IN)
- net at D31.2 (A): now also S31.4
- net at D36.2 (A): now also S36.4
- net at D22.2 (A): now also S22.4
- net at D33.2 (A): now also S33.4
- net at D13.2 (A): now also S13.4
- net at D19.2 (A): now also S19.4
- net at D6.2 (A): now also S6.4
- net at D2.2 (A): now also S2.4
- net at D30.2 (A): now also S30.4
- net at D18.2 (A): now also S18.4
- net at D29.2 (A): now also S29.4
- net at D21.2 (A): now also S21.4
- net at D27.2 (A): now also S27.4
- net at D9.2 (A): now also S9.4
- net at D3.2 (A): now also S3.4
- net at D10.2 (A): now also S8.4
- net at D20.2 (A): now also S20.4
- net at D5.2 (A): now also S11.4
- net at D7.2 (A): now also S5.4
- net at D28.2 (A): now also S28.4
- net at D4.2 (A): now also S4.4
- net at D17.2 (A): now also S17.4
- net at D32.2 (A): now also S32.4
- net at D24.2 (A): now also S24.4
- net at D26.2 (A): now also S26.4
- net at D34.2 (A): now also S34.4
- net at D25.2 (A): now also S25.4
- net at D12.2 (A): now also S10.4
- net at D15.2 (A): now also S15.4
- net at D23.2 (A): now also S23.4
- net at D16.2 (A): now also S16.4
- new net: D38.2 (A), S1.4
- no-connect marks 0 -> 72
Other:
- moved on the sheet: C2, R13, R14
