File: synthia/synthia.kicad_sch (KiCad schematic)
At the start: 90 parts, among them J1 MJ-63022B, J2 SJ3-35083C-TR, J3 PJ-007, J4 SDS-50J, Q1 IRF9540N, U1 TLV272IP, U2 STM32H750ZBT6, U3 LD1117V33, U4 PVA1EEH31.2NV2, U5 PVA1EEH31.2NV2

Commit message: Again did more Work on the PCB, Battery terminal is wired
Connections:
- no-connect marks 30 -> 90
Changed lines of the file:
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@@
+	)
+	(no_connect
+		(at 120.65 205.74)
+	)
+	(no_connect
+		(at 180.34 100.33)
+	)
+	(no_connect
+		(at 168.91 256.54)
 	)
 	(no_connect
@@
 	)
 	(no_connect
+		(at 153.67 256.54)
+	)
+	(no_connect
+		(at 187.96 100.33)
+	)
+	(no_connect
+		(at 171.45 256.54)
+	)
+	(no_connect
 		(at 77.47 59.69)
 	)
 	(no_connect
+		(at 130.81 256.54)
+	)
+	(no_connect
+		(at 135.89 205.74)
+	)
+	(no_connect
+		(at 107.95 256.54)
+	)
+	(no_connect
+		(at 128.27 205.74)
+	)
+	(no_connect
 		(at 36.83 127)
 	)
 	(no_connect
+		(at 186.69 256.54)
+	)
+	(no_connect
+		(at 146.05 205.74)
+	)
+	(no_connect
+		(at 151.13 205.74)
+	)
+	(no_connect
+		(at 106.68 100.33)
+	)
+	(no_connect
 		(at 129.54 95.25)
 	)
@@
 	)
 	(no_connect
+		(at 195.58 100.33)
+	)
+	(no_connect
+		(at 130.81 205.74)
+	)
+	(no_connect
+		(at 173.99 256.54)
+	)
+	(no_connect
 		(at 129.54 80.01)
 	)
 	(no_connect
+		(at 128.27 256.54)
+	)
+	(no_connect
+		(at 139.7 100.33)
+	)
+	(no_connect
 		(at 16.51 59.69)
 	)
 	(no_connect
+		(at 175.26 100.33)
+	)
+	(no_connect
+		(at 105.41 256.54)
+	)
+	(no_connect
 		(at 55.88 199.39)
 	)
 	(no_connect
+		(at 148.59 205.74)
+	)
+	(no_connect
+		(at 158.75 205.74)
+	)
+	(no_connect
 		(at 281.94 187.96)
 	)
 	(no_connect
+		(at 166.37 256.54)
+	)
+	(no_connect
+		(at 137.16 100.33)
+	)
+	(no_connect
+		(at 143.51 205.74)
+	)
+	(no_connect
 		(at 52.07 111.76)
 	)
 	(no_connect
+		(at 185.42 100.33)
+	)
+	(no_connect
+		(at 156.21 205.74)
+	)
+	(no_connect
 		(at 62.23 59.69)
 	)
@@
 	)
 	(no_connect
+		(at 148.59 256.54)
+	)
+	(no_connect
+		(at 129.54 100.33)
+	)
+	(no_connect
+		(at 125.73 205.74)
+	)
+	(no_connect
+		(at 176.53 256.54)
+	)
+	(no_connect
+		(at 127 100.33)
+	)
+	(no_connect
 		(at 46.99 59.69)
 	)
 	(no_connect
+		(at 193.04 100.33)
+	)
+	(no_connect
+		(at 156.21 256.54)
+	)
+	(no_connect
+		(at 177.8 100.33)
+	)
+	(no_connect
+		(at 132.08 100.33)
+	)
+	(no_connect
+		(at 133.35 205.74)
+	)
+	(no_connect
+		(at 144.78 100.33)
+	)
+	(no_connect
 		(at 21.59 111.76)
 	)
 	(no_connect
+		(at 140.97 256.54)
+	)
+	(no_connect
+		(at 118.11 256.54)
+	)
+	(no_connect
 		(at 73.66 158.75)
 	)
@@
 	)
 	(no_connect
+		(at 123.19 205.74)
+	)
+	(no_connect
+		(at 143.51 256.54)
+	)
+	(no_connect
 		(at 36.83 111.76)
 	)
 	(no_connect
+		(at 181.61 256.54)
+	)
+	(no_connect
+		(at 151.13 256.54)
+	)
+	(no_connect
+		(at 142.24 100.33)
+	)
+	(no_connect
 		(at 21.59 127)
 	)
@@
 	)
 	(no_connect
+		(at 190.5 100.33)
+	)
+	(no_connect
 		(at 55.88 158.75)
 	)
@@
 	)
 	(no_connect
+		(at 153.67 205.74)
+	)
+	(no_connect
 		(at 46.99 74.93)
 	)
@@
 	)
 	(no_connect
+		(at 111.76 100.33)
+	)
+	(no_connect
+		(at 109.22 100.33)
+	)
+	(no_connect
+		(at 113.03 205.74)
+	)
+	(no_connect
+		(at 124.46 100.33)
+	)
+	(no_connect
 		(at 67.31 127)
 	)
 	(no_connect
+		(at 147.32 100.33)
+	)
+	(no_connect
+		(at 123.19 256.54)
+	)
+	(no_connect
 		(at 77.47 74.93)
 	)
 	(no_connect
+		(at 138.43 256.54)
+	)
+	(no_connect
+		(at 146.05 256.54)
+	)
+	(no_connect
+		(at 120.65 256.54)
+	)
+	(no_connect
 		(at 73.66 199.39)
 	)
 	(no_connect
+		(at 184.15 256.54)
+	)
+	(no_connect
+		(at 163.83 256.54)
+	)
+	(no_connect
 		(at 110.49 205.74)
 	)
@@
 		(at 16.51 74.93)
 	)
+	(no_connect
+		(at 125.73 256.54)
+	)
 	(wire
