File: synthia/Synthia_DAC.kicad_sch (KiCad schematic)
At the start: 25 parts

Commit message: More updates to the Schematic, ports and solder points added for external components and were wired up
Parts:
- R15, R16, R17, R18, R19, R20, R21, R22, R23, R24, R25, R26, R27, R28, R29, R30, R31, R32, R33, R34, R35, R36, R37, R38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: footprint (none) -> Synthia_footprint_library:STA_CF14_STP
