File: synthia/synthia.kicad_pcb (KiCad board)
At the start: 2 copper layers, 0 parts

Commit message: Started on the PCB, button matrix is active
Parts:
- added D1: 1N4742A, Diode_THT:D_DO-41_SOD81_P10.16mm_Horizontal, F.Cu at (470.3, 161.7)
- added D10: 1N4001, Diode_THT:D_DO-41_SOD81_P10.16mm_Horizontal, F.Cu at (274.8, 298.0)
- added D11: 1N4001, Diode_THT:D_DO-41_SOD81_P10.16mm_Horizontal, F.Cu at (256.8, 318.0)
- added D12: 1N4001, Diode_THT:D_DO-41_SOD81_P10.16mm_Horizontal, F.Cu at (274.1, 277.8)
- added D13: 1N4001, Diode_THT:D_DO-41_SOD81_P10.16mm_Horizontal, F.Cu at (220.3, 298.0)
- added D14: 1N4001, Diode_THT:D_DO-41_SOD81_P10.16mm_Horizontal, F.Cu at (238.3, 298.0)
- added D15: 1N4001, Diode_THT:D_DO-41_SOD81_P10.16mm_Horizontal, F.Cu at (257.0, 298.0)
- added D16: 1N4001, Diode_THT:D_DO-41_SOD81_P10.16mm_Horizontal, F.Cu at (220.1, 277.8)
- added D17: 1N4001, Diode_THT:D_DO-41_SOD81_P10.16mm_Horizontal, F.Cu at (238.1, 277.8)
- added D18: 1N4001, Diode_THT:D_DO-41_SOD81_P10.16mm_Horizontal, F.Cu at (256.1, 277.8)
- added D19: 1N4001, Diode_THT:D_DO-41_SOD81_P10.16mm_Horizontal, F.Cu at (166.5, 318.0)
- added D2: 1N4001, Diode_THT:D_DO-41_SOD81_P10.16mm_Horizontal, F.Cu at (310.8, 298.0)
- added D20: 1N4001, Diode_THT:D_DO-41_SOD81_P10.16mm_Horizontal, F.Cu at (184.5, 318.0)
- added D21: 1N4001, Diode_THT:D_DO-41_SOD81_P10.16mm_Horizontal, F.Cu at (202.8, 318.0)
- added D22: 1N4001, Diode_THT:D_DO-41_SOD81_P10.16mm_Horizontal, F.Cu at (166.5, 298.0)
- added D23: 1N4001, Diode_THT:D_DO-41_SOD81_P10.16mm_Horizontal, F.Cu at (184.3, 298.0)
- added D24: 1N4001, Diode_THT:D_DO-41_SOD81_P10.16mm_Horizontal, F.Cu at (202.3, 298.0)
- added D25: 1N4001, Diode_THT:D_DO-41_SOD81_P10.16mm_Horizontal, F.Cu at (166.1, 277.8)
- added D26: 1N4001, Diode_THT:D_DO-41_SOD81_P10.16mm_Horizontal, F.Cu at (184.1, 277.8)
- added D27: 1N4001, Diode_THT:D_DO-41_SOD81_P10.16mm_Horizontal, F.Cu at (202.1, 277.8)
- added D28: 1N4001, Diode_THT:D_DO-41_SOD81_P10.16mm_Horizontal, F.Cu at (112.5, 318.0)
- added D29: 1N4001, Diode_THT:D_DO-41_SOD81_P10.16mm_Horizontal, F.Cu at (130.4, 318.0)
- added D3: 1N4001, Diode_THT:D_DO-41_SOD81_P10.16mm_Horizontal, F.Cu at (310.1, 277.8)
- added D30: 1N4001, Diode_THT:D_DO-41_SOD81_P10.16mm_Horizontal, F.Cu at (148.3, 318.0)
- added D31: 1N4001, Diode_THT:D_DO-41_SOD81_P10.16mm_Horizontal, F.Cu at (112.3, 298.0)
- added D32: 1N4001, Diode_THT:D_DO-41_SOD81_P10.16mm_Horizontal, F.Cu at (130.5, 298.0)
- added D33: 1N4001, Diode_THT:D_DO-41_SOD81_P10.16mm_Horizontal, F.Cu at (148.3, 298.0)
- added D34: 1N4001, Diode_THT:D_DO-41_SOD81_P10.16mm_Horizontal, F.Cu at (112.3, 278.0)
- added D35: 1N4001, Diode_THT:D_DO-41_SOD81_P10.16mm_Horizontal, F.Cu at (130.2, 278.0)
- added D36: 1N4001, Diode_THT:D_DO-41_SOD81_P10.16mm_Horizontal, F.Cu at (148.1, 277.8)
- added D38: 1N4001, Diode_THT:D_DO-41_SOD81_P10.16mm_Horizontal, F.Cu at (311.0, 318.0)
- added D4: 1N4001, Diode_THT:D_DO-41_SOD81_P10.16mm_Horizontal, F.Cu at (292.8, 318.0)
- added D5: 1N4001, Diode_THT:D_DO-41_SOD81_P10.16mm_Horizontal, F.Cu at (293.0, 298.0)
- added D6: 1N4001, Diode_THT:D_DO-41_SOD81_P10.16mm_Horizontal, F.Cu at (292.1, 277.8)
- added D7: 1N4001, Diode_THT:D_DO-41_SOD81_P10.16mm_Horizontal, F.Cu at (220.5, 318.0)
- added D8: 1N4001, Diode_THT:D_DO-41_SOD81_P10.16mm_Horizontal, F.Cu at (274.8, 318.0)
- added D9: 1N4001, Diode_THT:D_DO-41_SOD81_P10.16mm_Horizontal, F.Cu at (238.5, 318.0)
- added Q1: IRF9540N, Package_TO_SOT_THT:TO-220-3_Vertical, F.Cu at (471.6, 173.4)
- added Q2: L78M05CV, Synthia_footprint_library:TO254P450X1020X1935-3P, F.Cu at (476.7, 166.1)
- added S1: TL1105BF160Q, Synthia_footprint_library:SW_TL1105BF160Q, F.Cu at (318.0, 324.0)
- added S10: TL1105BF160Q, Synthia_footprint_library:SW_TL1105BF160Q, F.Cu at (281.2, 286.0)
- added S11: TL1105BF160Q, Synthia_footprint_library:SW_TL1105BF160Q, F.Cu at (300.0, 306.0)
- added S12: TL1105BF160Q, Synthia_footprint_library:SW_TL1105BF160Q, F.Cu at (264.0, 324.5)
- added S13: TL1105BF160Q, Synthia_footprint_library:SW_TL1105BF160Q, F.Cu at (227.5, 305.5)
- added S14: TL1105BF160Q, Synthia_footprint_library:SW_TL1105BF160Q, F.Cu at (245.5, 305.8)
- added S15: TL1105BF160Q, Synthia_footprint_library:SW_TL1105BF160Q, F.Cu at (264.2, 306.0)
- added S16: TL1105BF160Q, Synthia_footprint_library:SW_TL1105BF160Q, F.Cu at (227.2, 285.8)
- added S17: TL1105BF160Q, Synthia_footprint_library:SW_TL1105BF160Q, F.Cu at (245.2, 285.8)
- added S18: TL1105BF160Q, Synthia_footprint_library:SW_TL1105BF160Q, F.Cu at (263.5, 286.0)
- added S19: TL1105BF160Q, Synthia_footprint_library:SW_TL1105BF160Q, F.Cu at (173.7, 325.0)
- added S2: TL1105BF160Q, Synthia_footprint_library:SW_TL1105BF160Q, F.Cu at (318.0, 306.0)
- added S20: TL1105BF160Q, Synthia_footprint_library:SW_TL1105BF160Q, F.Cu at (191.7, 325.0)
- added S21: TL1105BF160Q, Synthia_footprint_library:SW_TL1105BF160Q, F.Cu at (210.2, 324.8)
- added S22: TL1105BF160Q, Synthia_footprint_library:SW_TL1105BF160Q, F.Cu at (173.7, 305.5)
- added S23: TL1105BF160Q, Synthia_footprint_library:SW_TL1105BF160Q, F.Cu at (191.5, 305.5)
- added S24: TL1105BF160Q, Synthia_footprint_library:SW_TL1105BF160Q, F.Cu at (209.5, 305.5)
- added S25: TL1105BF160Q, Synthia_footprint_library:SW_TL1105BF160Q, F.Cu at (173.2, 285.8)
- added S26: TL1105BF160Q, Synthia_footprint_library:SW_TL1105BF160Q, F.Cu at (191.2, 285.8)
- added S27: TL1105BF160Q, Synthia_footprint_library:SW_TL1105BF160Q, F.Cu at (209.2, 285.8)
- added S28: TL1105BF160Q, Synthia_footprint_library:SW_TL1105BF160Q, F.Cu at (119.9, 325.2)
- added S29: TL1105BF160Q, Synthia_footprint_library:SW_TL1105BF160Q, F.Cu at (137.7, 325.0)
- added S3: TL1105BF160Q, Synthia_footprint_library:SW_TL1105BF160Q, F.Cu at (317.2, 286.2)
- added S30: TL1105BF160Q, Synthia_footprint_library:SW_TL1105BF160Q, F.Cu at (155.7, 325.0)
- added S31: TL1105BF160Q, Synthia_footprint_library:SW_TL1105BF160Q, F.Cu at (119.5, 305.5)
- added S32: TL1105BF160Q, Synthia_footprint_library:SW_TL1105BF160Q, F.Cu at (137.7, 305.5)
- added S33: TL1105BF160Q, Synthia_footprint_library:SW_TL1105BF160Q, F.Cu at (155.5, 305.5)
- added S34: TL1105BF160Q, Synthia_footprint_library:SW_TL1105BF160Q, F.Cu at (119.5, 285.5)
- added S35: TL1105BF160Q, Synthia_footprint_library:SW_TL1105BF160Q, F.Cu at (137.2, 285.5)
- added S36: TL1105BF160Q, Synthia_footprint_library:SW_TL1105BF160Q, F.Cu at (155.2, 285.8)
- added S4: TL1105BF160Q, Synthia_footprint_library:SW_TL1105BF160Q, F.Cu at (300.0, 324.2)
- added S5: TL1105BF160Q, Synthia_footprint_library:SW_TL1105BF160Q, F.Cu at (227.7, 324.5)
- added S6: TL1105BF160Q, Synthia_footprint_library:SW_TL1105BF160Q, F.Cu at (299.2, 286.2)
- added S7: TL1105BF160Q, Synthia_footprint_library:SW_TL1105BF160Q, F.Cu at (282.0, 324.5)
- added S8: TL1105BF160Q, Synthia_footprint_library:SW_TL1105BF160Q, F.Cu at (282.0, 306.0)
- added S9: TL1105BF160Q, Synthia_footprint_library:SW_TL1105BF160Q, F.Cu at (245.7, 324.5)
Other:
- board outline added: 271 x 227 mm

Commit message: More PCB Updates for the Matrix
Parts:
- moved D11 27.9 mm to (284.4, 313.8)
- moved D8 27.9 mm to (302.4, 313.8)
- moved D19 27.9 mm to (194.1, 313.8)
- moved D20 27.9 mm to (212.1, 313.8)
- moved D21 27.9 mm to (230.3, 313.8)
- moved D28 27.9 mm to (140.1, 313.8)
- moved D29 27.9 mm to (158.0, 313.8)
- moved D7 27.9 mm to (248.1, 313.8)
- moved S19 27.9 mm to (201.2, 320.8)
- moved S20 27.9 mm to (219.2, 320.8)
- moved S21 27.9 mm to (237.8, 320.5)
- moved S28 27.9 mm to (147.5, 321.0)
- moved S29 27.9 mm to (165.2, 320.8)
- moved S30 27.9 mm to (183.2, 320.8)
- moved S5 27.9 mm to (255.2, 320.2)
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Other:
- board size 271 x 227 mm -> 291 x 258.5 mm

Commit message: More updates to the Schematic, implemented some of the ports that will be on the pcb
Parts:
- moved Q2 185.5 mm to (292.1, 183.4)
- moved D1 178.6 mm to (292.0, 172.5)
- moved Q1 164.8 mm to (307.0, 178.9)
Other:
- board size 291 x 258.5 mm -> 285 x 257.5 mm
Changed lines of the file:
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@@
 	(footprint "Synthia_footprint_library:TO254P450X1020X1935-3P"
 		(layer "F.Cu")
-		(at 476.7382 166.1138)
+		(at 292.08 183.4078)
 		(property "Reference" "Q2"
 			(at -1.987805 -3.822735 0)
@@
 	(footprint "Package_TO_SOT_THT:TO-220-3_Vertical"
 		(layer "F.Cu")
-		(at 471.65 173.45)
+		(at 306.96 178.95)
 		(descr "TO-220-3, Vertical, RM 2.54mm, see https://www.vishay.com/docs/66542/to-220-1.pdf, generated with kicad-footprint-generator TO_SOT_THT_generate.py")
 		(tags "TO-220-3 Vertical RM 2.54mm")
@@
 	(footprint "Diode_THT:D_DO-41_SOD81_P10.16mm_Horizontal"
 		(layer "F.Cu")
-		(at 470.29 161.66)
+		(at 292 172.5)
 		(descr "Diode, DO-41_SOD81 series, Axial, Horizontal, pin pitch=10.16mm, length*diameter=5.2*2.7mm^2, https://www.diodes.com/assets/Package-Files/DO-41-Plastic.pdf")
 		(tags "Diode DO-41_SOD81 series Axial Horizontal pin pitch 10.16mm  length 5.2mm diameter 2.7mm")
@@
 		(embedded_fonts no)
 	)
-	(gr_rect
-		(start 199.86 110.41)
-		(end 221.75 119.6)
-		(stroke
-			(width 0.2)
-			(type default)
-		)
-		(fill no)
-		(layer "F.Cu")
-	)
-	(gr_circle
-		(center 193.019769 247)
-		(end 117.019769 323)
+	(gr_line
+		(start 75.5 205)
+		(end -86.5 205)
 		(stroke
 			(width 0.2)
 			(type default)
 		)
-		(fill no)
 		(layer "B.Cu")
 	)
 	(gr_line
-		(start 75.5 205)
-		(end -86.5 205)
+		(start 370.5 90.275)
+		(end 160.967045 147.015676)
 		(stroke
-			(width 0.2)
+			(width 0.05)
 			(type default)
 		)
-		(layer "B.Cu")
+		(layer "Edge.Cuts")
 	)
 	(gr_line
-		(start 356.5 226)
-		(end 376.52907 354.455601)
+		(start 370.5 347.725)
+		(end 370.5 90.275)
 		(stroke
-			(width 0.2)
+			(width 0.05)
 			(type default)
 		)
-		(layer "B.Cu")
+		(layer "Edge.Cuts")
 	)
-	(gr_rect
-		(start 85.5 96)
-		(end 376.5 354.5)
+	(gr_arc
+		(start 187.625 347.725)
+		(mid 86.389039 259.04603)
+		(end 160.967046 147.015676)
 		(stroke
 			(width 0.05)
 			(type default)
 		)
-		(fill no)
 		(layer "Edge.Cuts")
 	)
 	(gr_line
-		(start 376.5 226)
-		(end 85.5 226)
+		(start 370.5 347.725)
+		(end 187.625 347.725)
 		(stroke
 			(width 0.05)

Commit message: More updates to Schematic, added latching switch as a symbol and footprint
Parts:
- removed Q2: L78M05CV, Synthia_footprint_library:TO254P450X1020X1935-3P
- added C1: 100 nF, Capacitor_THT:CP_Radial_Tantal_D5.0mm_P5.00mm, F.Cu at (170.5, 81.5)
- added C2: 10 uF, Capacitor_THT:CP_Radial_Tantal_D5.0mm_P5.00mm, F.Cu at (170.2, 62.7)
- added C3: 500 uF, Capacitor_THT:CP_Radial_Tantal_D5.0mm_P5.00mm, F.Cu at (170.2, 71.2)
- added J1: MJ-63022B, Synthia_footprint_library:CUI_MJ-63022B, F.Cu at (193.7, 94.6)
- added J2: SJ3-35083C-TR, Synthia_footprint_library:SAMESKY_SJ3-35083C-TR, F.Cu at (221.9, 74.6)
- added J3: PJ-007, Synthia_footprint_library:SAMESKY_PJ-007, F.Cu at (223.3, 109.3)
- added J4: SDS-50J, Synthia_footprint_library:CUI_SDS-50J, F.Cu at (205.8, 136.6)
- added R10: 100k, Synthia_footprint_library:STA_CF14_STP, F.Cu at (157.0, 330.0)
- added R11: 100k, Synthia_footprint_library:STA_CF14_STP, F.Cu at (175.1, 330.0)
- added R13: 100k, Synthia_footprint_library:STA_CF14_STP, F.Cu at (319.1, 330.0)
- added R14: 100k, Synthia_footprint_library:STA_CF14_STP, F.Cu at (337.6, 330.0)
- added R15: 100k, Synthia_footprint_library:STA_CF14_STP, F.Cu at (153.3, 149.0)
- added R16: 100k, Synthia_footprint_library:STA_CF14_STP, F.Cu at (153.3, 153.3)
- added R17: 100k, Synthia_footprint_library:STA_CF14_STP, F.Cu at (153.3, 157.6)
- added R18: 100k, Synthia_footprint_library:STA_CF14_STP, F.Cu at (153.3, 161.8)
- added R19: 100k, Synthia_footprint_library:STA_CF14_STP, F.Cu at (153.3, 166.1)
- added R2: 100k, Synthia_footprint_library:STA_CF14_STP, F.Cu at (153.3, 68.5)
- added R20: 100k, Synthia_footprint_library:STA_CF14_STP, F.Cu at (153.3, 170.4)
- added R21: 100k, Synthia_footprint_library:STA_CF14_STP, F.Cu at (153.3, 174.7)
- added R22: 100k, Synthia_footprint_library:STA_CF14_STP, F.Cu at (153.3, 178.9)
- added R23: 100k, Synthia_footprint_library:STA_CF14_STP, F.Cu at (153.3, 183.2)
- added R24: 100k, Synthia_footprint_library:STA_CF14_STP, F.Cu at (167.8, 149.0)
- added R25: 100k, Synthia_footprint_library:STA_CF14_STP, F.Cu at (167.8, 153.3)
- added R26: 100k, Synthia_footprint_library:STA_CF14_STP, F.Cu at (167.8, 157.6)
- added R27: 100k, Synthia_footprint_library:STA_CF14_STP, F.Cu at (167.8, 161.8)
- added R28: 100k, Synthia_footprint_library:STA_CF14_STP, F.Cu at (167.8, 166.1)
- added R29: 100k, Synthia_footprint_library:STA_CF14_STP, F.Cu at (167.8, 170.4)
- added R3: 100k, Synthia_footprint_library:STA_CF14_STP, F.Cu at (247.0, 330.0)
- added R30: 100k, Synthia_footprint_library:STA_CF14_STP, F.Cu at (167.8, 174.7)
- added R31: 100k, Synthia_footprint_library:STA_CF14_STP, F.Cu at (167.8, 178.9)
- added R32: 100k, Synthia_footprint_library:STA_CF14_STP, F.Cu at (167.8, 183.2)
- added R33: 100k, Synthia_footprint_library:STA_CF14_STP, F.Cu at (182.3, 149.0)
- added R34: 100k, Synthia_footprint_library:STA_CF14_STP, F.Cu at (182.3, 153.3)
- added R35: 100k, Synthia_footprint_library:STA_CF14_STP, F.Cu at (182.3, 157.6)
- added R36: 100k, Synthia_footprint_library:STA_CF14_STP, F.Cu at (182.3, 161.8)
- added R37: 100k, Synthia_footprint_library:STA_CF14_STP, F.Cu at (182.3, 166.1)
- added R38: 100k, Synthia_footprint_library:STA_CF14_STP, F.Cu at (182.3, 170.4)
- added R39: 100k, Synthia_footprint_library:STA_CF14_STP, F.Cu at (182.3, 174.7)
- added R4: 100k, Synthia_footprint_library:STA_CF14_STP, F.Cu at (265.1, 330.0)
- added R40: 100k, Synthia_footprint_library:STA_CF14_STP, F.Cu at (301.1, 330.0)
- added R5: 100k, Synthia_footprint_library:STA_CF14_STP, F.Cu at (283.1, 330.0)
- added R50: P120PK-Y25BR10K, Synthia_footprint_library:POT_P120PK-x25_TTE, F.Cu at (189.3, 83.4)
- added R51: 100k, Synthia_footprint_library:STA_CF14_STP, F.Cu at (153.3, 72.8)
- added R52: 100k, Synthia_footprint_library:STA_CF14_STP, F.Cu at (153.3, 77.0)
- added R53: 100k, Synthia_footprint_library:STA_CF14_STP, F.Cu at (153.3, 81.3)
- added R54: 100k, Synthia_footprint_library:STA_CF14_STP, F.Cu at (153.3, 85.6)
- added R55: 100k, Synthia_footprint_library:STA_CF14_STP, F.Cu at (153.3, 89.9)
- added R56: 100k, Synthia_footprint_library:STA_CF14_STP, F.Cu at (153.3, 94.1)
- added R57: 100k, Synthia_footprint_library:STA_CF14_STP, F.Cu at (153.3, 98.4)
- added R58: 100k, Synthia_footprint_library:STA_CF14_STP, F.Cu at (153.3, 102.7)
- added R59: 100k, Synthia_footprint_library:STA_CF14_STP, F.Cu at (153.3, 107.0)
- added R6: 100k, Synthia_footprint_library:STA_CF14_STP, F.Cu at (193.1, 330.0)
- added R60: 100k, Synthia_footprint_library:STA_CF14_STP, F.Cu at (153.3, 111.3)
- added R61: 100k, Synthia_footprint_library:STA_CF14_STP, F.Cu at (153.3, 115.5)
- added R62: 100k, Synthia_footprint_library:STA_CF14_STP, F.Cu at (153.3, 119.8)
- added R63: 100k, Synthia_footprint_library:STA_CF14_STP, F.Cu at (153.3, 124.1)
- added R64: 100k, Synthia_footprint_library:STA_CF14_STP, F.Cu at (153.3, 128.4)
- added R7: 100k, Synthia_footprint_library:STA_CF14_STP, F.Cu at (211.1, 330.0)
- added R8: 100k, Synthia_footprint_library:STA_CF14_STP, F.Cu at (229.1, 330.0)
- added R9: 100k, Synthia_footprint_library:STA_CF14_STP, F.Cu at (139.1, 330.0)
- added S37: TL1105BF160Q, Synthia_footprint_library:SW_TL1105BF160Q, F.Cu at (171.7, 90.2)
- added S38: TL1105BF160Q, Synthia_footprint_library:SW_TL1105BF160Q, F.Cu at (171.7, 97.8)
- added S39: TL1105BF160Q, Synthia_footprint_library:SW_TL1105BF160Q, F.Cu at (171.7, 105.3)
- added S40: TL1105BF160Q, Synthia_footprint_library:SW_TL1105BF160Q, F.Cu at (171.7, 112.9)
- added S41: TL1105BF160Q, Synthia_footprint_library:SW_TL1105BF160Q, F.Cu at (171.7, 120.4)
- added TP1: Speaker, TestPoint:TestPoint_Plated_Hole_D2.0mm, F.Cu at (178.8, 104.7)
- added TP10: StrumPad Pin #1, TestPoint:TestPoint_Plated_Hole_D2.0mm, F.Cu at (183.4, 109.4)
- added TP11: StrumPad Pin #2, TestPoint:TestPoint_Plated_Hole_D2.0mm, F.Cu at (183.4, 114.0)
- added TP12: StrumPad Pin #3, TestPoint:TestPoint_Plated_Hole_D2.0mm, F.Cu at (183.4, 118.7)
- added TP13: Switch Pin #1, TestPoint:TestPoint_Plated_Hole_D2.0mm, F.Cu at (183.4, 123.3)
- added TP14: Switch Pin #2, TestPoint:TestPoint_Plated_Hole_D2.0mm, F.Cu at (183.4, 128.0)
- added TP15: Speaker GND, TestPoint:TestPoint_Plated_Hole_D2.0mm, F.Cu at (188.1, 104.7)
- added TP16: Shield / Ground, TestPoint:TestPoint_Plated_Hole_D2.0mm, F.Cu at (188.1, 109.4)
- added TP17: Sink, TestPoint:TestPoint_Plated_Hole_D2.0mm, F.Cu at (188.1, 114.0)
- added TP18: Source, TestPoint:TestPoint_Plated_Hole_D2.0mm, F.Cu at (188.1, 118.7)
- added TP19: MicroUSB Pin #1, TestPoint:TestPoint_Plated_Hole_D2.0mm, F.Cu at (188.1, 123.3)
- added TP2: +9V, TestPoint:TestPoint_Pad_2.0x2.0mm, F.Cu at (178.5, 138.4)
- added TP20: MicroUSB Pin #2, TestPoint:TestPoint_Plated_Hole_D2.0mm, F.Cu at (188.1, 128.0)
- added TP21: MicroUSB Pin #3, TestPoint:TestPoint_Plated_Hole_D2.0mm, F.Cu at (192.7, 104.7)
- added TP22: MicroUSB Pin #4, TestPoint:TestPoint_Plated_Hole_D2.0mm, F.Cu at (192.7, 109.4)
- added TP23: MicroUSB Pin #5, TestPoint:TestPoint_Plated_Hole_D2.0mm, F.Cu at (192.7, 114.0)
- added TP3: +3.3V, TestPoint:TestPoint_Pad_2.0x2.0mm, F.Cu at (178.5, 142.4)
- added TP4: Battery_2, TestPoint:TestPoint_Plated_Hole_D2.0mm, F.Cu at (178.8, 109.4)
- added TP5: Battery_3, TestPoint:TestPoint_Plated_Hole_D2.0mm, F.Cu at (178.8, 114.0)
- added TP6: Battery_1, TestPoint:TestPoint_Plated_Hole_D2.0mm, F.Cu at (178.8, 118.7)
- added TP7: Battery_1_GND, TestPoint:TestPoint_Plated_Hole_D2.0mm, F.Cu at (178.8, 123.3)
- added TP8: Battery_2_GND, TestPoint:TestPoint_Plated_Hole_D2.0mm, F.Cu at (178.8, 128.0)
- added TP9: Battery_3_GND, TestPoint:TestPoint_Plated_Hole_D2.0mm, F.Cu at (183.4, 104.7)
- added U1: TLV272IP, Synthia_footprint_library:DIP794W45P254L959H508Q8, F.Cu at (206.5, 76.0)
- added U2: STM32H750ZBT6, Synthia_footprint_library:LQFP144_STM, F.Cu at (207.5, 114.9)
- added U3: LD1117V33, Synthia_footprint_library:TO255P1020X450X1968-3, F.Cu at (165.5, 136.0)
- moved S15 1.13 mm to (272.9, 294.6)
- moved D31 1.13 mm to (121.1, 286.6)
- moved D34 1.13 mm to (103.8, 258.4)
- moved D35 1.13 mm to (121.7, 258.4)
- moved S34 1.13 mm to (111.0, 265.9)
- moved D10 1.13 mm to (283.6, 286.6)
- moved D11 1.13 mm to (283.7, 314.6)
- moved D12 1.13 mm to (265.6, 258.1)
- moved D13 1.13 mm to (229.1, 286.6)
- moved D14 1.13 mm to (247.1, 286.6)
- moved D15 1.13 mm to (265.8, 286.6)
- moved D16 1.13 mm to (211.6, 258.1)
- moved D17 1.13 mm to (229.6, 258.1)
- moved D18 1.13 mm to (247.6, 258.1)
- moved D19 1.13 mm to (193.3, 314.6)
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Connections:
- Q1 pad 2: +9V -> Net-(Q1-D)
Other:
- copper layers 2 -> 4
