File: synthia/synthia.kicad_pcb (KiCad board)
At the start: 2 copper layers, 300 x 271.1 mm, 229 parts, among them J1 MJ-63022B, J2 SJ3-35083C-TR, J3 PJ-007, J4 SDS-50J, Q1 IRF9540N, U1 TLV272IP, U2 STM32H750ZBT6, U3 LD1117V33, U4 PVA1EEH31.2NV2, U5 PVA1EEH31.2NV2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

Commit message: Scaled down the PCB to be able to fit inside the 3 model case
Parts:
- moved R79 19.0 mm to (177.8, 179.0)
- moved LOGO 16.8 mm to (369.2, 319.8)
Other:
- board size 300 x 271.1 mm -> 282.4 x 255.2 mm
Changed lines of the file:
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@@
 	(footprint "Synthia_footprint_library:POT_P120PK-x25_TTE"
 		(layer "F.Cu")
-		(at 167.50925 162.9409)
+		(at 177.75425 178.9677)
 		(tags "P120PK-Y25BR10K ")
 		(property "Reference" "R79"
@@
 	(footprint "LOGO"
 		(layer "F.Cu")
-		(at 373.67 335.98)
+		(at 369.16 319.81)
 		(property "Reference" "LOGO"
 			(at 0 0 0)
@@
 	(gr_line
 		(start 241.782488 124.84112)
-		(end 246.740566 123.510616)
+		(end 246.666174 123.530579)
 		(stroke
 			(width 0.1)
@@
 	)
 	(gr_line
-		(start 251.549526 122.220127)
+		(start 251.623377 122.200309)
 		(end 272.53 116.59)
 		(stroke
@@
 	)
 	(gr_arc
-		(start 203.343931 354.009955)
-		(mid 96.480915 260.325678)
-		(end 175.375179 142.121857)
+		(start 214.326764 337.990435)
+		(mid 113.735931 249.804834)
+		(end 187.999601 138.538835)
 		(stroke
-			(width 0.05)
+			(width 0.047065)
 			(type default)
 		)
@@
 	)
 	(gr_line
-		(start 395.597075 82.93)
-		(end 175.38 142.121857)
+		(start 395.295862 82.821164)
+		(end 188.004137 138.538835)
 		(stroke
-			(width 0.05)
+			(width 0.047065)
 			(type default)
 		)
@@
 	)
 	(gr_line
-		(start 395.597075 353.85)
-		(end 203.34 354.01)
+		(start 395.295862 337.839872)
+		(end 214.323063 337.990478)
 		(stroke
-			(width 0.05)
+			(width 0.047065)
 			(type default)
 		)
@@
 	)
 	(gr_line
-		(start 395.597075 353.85)
-		(end 395.597075 82.929123)
+		(start 395.295862 337.839872)
+		(end 395.295862 82.820341)
 		(stroke
-			(width 0.05)
+			(width 0.047065)
 			(type default)
 		)
@@
 	)
 	(gr_text "REV 1.0"
-		(at 357.46 352.41 0)
+		(at 352.95 336.24 0)
 		(layer "F.SilkS")
 		(effects

Commit message: made 3D model of current PCB, will likely be updated and replaced when needed
Parts:
- moved R79 8.05 mm to (171.4, 183.9)
Connections:
- R52 pad 2: Net-(R52-Pad2) -> Net-(U2A-PB1)
- R64 pad 2: Net-(R52-Pad2) -> Net-(U2A-PB1)
- R66 pad 2: Net-(R66-Pad2) -> Net-(U2A-PC5)
- R67 pad 1: Net-(R66-Pad2) -> Net-(U2A-PC5)
- R79 pad 2: unconnected-(R79-Pad2) -> Net-(U2A-PA7)
- U2 pad 43: unconnected-(U2A-PA7-Pad43) -> Net-(U2A-PA7)
- U2 pad 44: unconnected-(U2A-PC4-Pad44) -> Net-(U2A-PC4)
- U2 pad 45: unconnected-(U2A-PC5-Pad45) -> Net-(U2A-PC5)
- U2 pad 46: unconnected-(U2A-PB0-Pad46) -> Net-(U2A-PB0)
- U2 pad 47: unconnected-(U2A-PB1-Pad47) -> Net-(U2A-PB1)
- U4 pad 4: unconnected-(U4-Pad4) -> Net-(U2A-PB0)
- U5 pad 3: unconnected-(U5-Pad3) -> Net-(U2A-PC4)
Routing:
- net Net-(U2A-PB1): track 0.00 -> 14.2 mm
- net Net-(R52-Pad2): track 14.2 -> 0.00 mm
- net Net-(U2A-PC5): track 0.00 -> 11.8 mm
- net Net-(R66-Pad2): track 11.8 -> 0.00 mm
- net GND: vias 43 -> 42
Changed lines of the file:
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@@
 			(net "unconnected-(U2A-PA3-Pad37)")
 			(pinfunction "PA3_37")
-			(pintype "bidirectional")
+			(pintype "bidirectional+no_connect")
 		)
 		(pad "38" smd rect
@@
 			(net "unconnected-(U2A-PA4-Pad40)")
 			(pinfunction "PA4_40")
-			(pintype "bidirectional")
+			(pintype "bidirectional+no_connect")
 		)
 		(pad "41" smd rect
@@
 			(net "unconnected-(U2A-PA5-Pad41)")
 			(pinfunction "PA5_41")
-			(pintype "bidirectional")
+			(pintype "bidirectional+no_connect")
 		)
 		(pad "42" smd rect
@@
 			(net "unconnected-(U2A-PA6-Pad42)")
 			(pinfunction "PA6_42")
-			(pintype "bidirectional")
+			(pintype "bidirectional+no_connect")
 		)
 		(pad "43" smd rect
@@
 			(size 0.2794 1.3589)
 			(layers "F.Cu" "F.Mask" "F.Paste")
-			(net "unconnected-(U2A-PA7-Pad43)")
+			(net "Net-(U2A-PA7)")
 			(pinfunction "PA7_43")
 			(pintype "bidirectional")
@@
 			(size 0.2794 1.3589)
 			(layers "F.Cu" "F.Mask" "F.Paste")
-			(net "unconnected-(U2A-PC4-Pad44)")
+			(net "Net-(U2A-PC4)")
 			(pinfunction "PC4_44")
 			(pintype "bidirectional")
@@
 			(size 0.2794 1.3589)
 			(layers "F.Cu" "F.Mask" "F.Paste")
-			(net "unconnected-(U2A-PC5-Pad45)")
+			(net "Net-(U2A-PC5)")
 			(pinfunction "PC5_45")
 			(pintype "bidirectional")
@@
 			(size 0.2794 1.3589)
 			(layers "F.Cu" "F.Mask" "F.Paste")
-			(net "unconnected-(U2A-PB0-Pad46)")
+			(net "Net-(U2A-PB0)")
 			(pinfunction "PB0_46")
 			(pintype "bidirectional")
@@
 			(size 0.2794 1.3589)
 			(layers "F.Cu" "F.Mask" "F.Paste")
-			(net "unconnected-(U2A-PB1-Pad47)")
+			(net "Net-(U2A-PB1)")
 			(pinfunction "PB1_47")
 			(pintype "bidirectional")
@@
 			(net "unconnected-(U2A-PB2-Pad48)")
 			(pinfunction "PB2_48")
-			(pintype "bidirectional")
+			(pintype "bidirectional+no_connect")
 		)
 		(pad "49" smd rect
@@
 			(net "unconnected-(U2A-PF11-Pad49)")
 			(pinfunction "PF11_49")
-			(pintype "bidirectional")
+			(pintype "bidirectional+no_connect")
 		)
 		(pad "50" smd rect
@@
 			(net "unconnected-(U2A-PF12-Pad50)")
 			(pinfunction "PF12_50")
-			(pintype "bidirectional")
+			(pintype "bidirectional+no_connect")
 		)
 		(pad "51" smd rect
@@
 			(net "unconnected-(U2A-PF13-Pad53)")
 			(pinfunction "PF13_53")
-			(pintype "bidirectional")
+			(pintype "bidirectional+no_connect")
 		)
 		(pad "54" smd rect
@@
 			(net "unconnected-(U2A-PF14-Pad54)")
 			(pinfunction "PF14_54")
-			(pintype "bidirectional")
+			(pintype "bidirectional+no_connect")
 		)
 		(pad "55" smd rect
@@
 			(net "unconnected-(U2A-PF15-Pad55)")
 			(pinfunction "PF15_55")
-			(pintype "bidirectional")
+			(pintype "bidirectional+no_connect")
 		)
 		(pad "56" smd rect
@@
 			(net "unconnected-(U2A-PG0-Pad56)")
 			(pinfunction "PG0_56")
-			(pintype "bidirectional")
+			(pintype "bidirectional+no_connect")
 		)
 		(pad "57" smd rect
@@
 			(net "unconnected-(U2A-PG1-Pad57)")
 			(pinfunction "PG1_57")
-			(pintype "bidirectional")
+			(pintype "bidirectional+no_connect")
 		)
 		(pad "58" smd rect
@@
 			(net "unconnected-(U2A-PE7-Pad58)")
 			(pinfunction "PE7_58")
-			(pintype "bidirectional")
+			(pintype "bidirectional+no_connect")
 		)
 		(pad "59" smd rect
@@
 			(net "unconnected-(U2A-PE8-Pad59)")
 			(pinfunction "PE8_59")
-			(pintype "bidirectional")
+			(pintype "bidirectional+no_connect")
 		)
 		(pad "60" smd rect
@@
 			(net "unconnected-(U2A-PE9-Pad60)")
 			(pinfunction "PE9_60")
-			(pintype "bidirectional")
+			(pintype "bidirectional+no_connect")
 		)
 		(pad "61" smd rect
@@
 			(net "unconnected-(U2A-PE10-Pad63)")
 			(pinfunction "PE10_63")
-			(pintype "bidirectional")
+			(pintype "bidirectional+no_connect")
 		)
 		(pad "64" smd rect
@@
 			(net "unconnected-(U2A-PE11-Pad64)")
 			(pinfunction "PE11_64")
-			(pintype "bidirectional")
+			(pintype "bidirectional+no_connect")
 		)
 		(pad "65" smd rect
@@
 			(net "unconnected-(U2A-PE12-Pad65)")
 			(pinfunction "PE12_65")
-			(pintype "bidirectional")
+			(pintype "bidirectional+no_connect")
 		)
 		(pad "66" smd rect
@@
 			(net "unconnected-(U2A-PE13-Pad66)")
 			(pinfunction "PE13_66")
-			(pintype "bidirectional")
+			(pintype "bidirectional+no_connect")
 		)
 		(pad "67" smd rect
@@
 			(net "unconnected-(U2A-PE14-Pad67)")
 			(pinfunction "PE14_67")
-			(pintype "bidirectional")
+			(pintype "bidirectional+no_connect")
 		)
 		(pad "68" smd rect
@@
 			(net "unconnected-(U2A-PE15-Pad68)")
 			(pinfunction "PE15_68")
-			(pintype "bidirectional")
+			(pintype "bidirectional+no_connect")
 		)
 		(pad "69" smd rect
@@
 			(net "unconnected-(U2A-PB10-Pad69)")
 			(pinfunction "PB10_69")
-			(pintype "bidirectional")
+			(pintype "bidirectional+no_connect")
 		)
 		(pad "70" smd rect
@@
 			(net "unconnected-(U2A-PB11-Pad70)")
 			(pinfunction "PB11_70")
-			(pintype "bidirectional")
+			(pintype "bidirectional+no_connect")
 		)
 		(pad "71" smd rect
@@
 			(layers "*.Cu" "*.Mask")
 			(remove_unused_layers no)
-			(net "unconnected-(U4-Pad4)")
+			(net "Net-(U2A-PB0)")
 			(pinfunction "4_4")
 			(pintype "unspecified")
@@
 			(layers "*.Cu" "*.Mask")
 			(remove_unused_layers no)
-			(net "Net-(R52-Pad2)")
+			(net "Net-(U2A-PB1)")
 			(pintype "passive")
 		)
@@
 			(layers "*.Cu" "*.Mask")
 			(remove_unused_layers no)
-			(net "Net-(R66-Pad2)")
+			(net "Net-(U2A-PC5)")
 			(pintype "passive")
 		)
@@
 			(layers "*.Cu" "*.Mask")
 			(remove_unused_layers no)
-			(net "Net-(R52-Pad2)")
+			(net "Net-(U2A-PB1)")
 			(pintype "passive")
 		)
@@
 			(layers "*.Cu" "*.Mask")
 			(remove_unused_layers no)
-			(net "unconnected-(U5-Pad3)")
+			(net "Net-(U2A-PC4)")
 			(pinfunction "3_3")
 			(pintype "unspecified")
@@
 	(footprint "Synthia_footprint_library:POT_P120PK-x25_TTE"
 		(layer "F.Cu")
-		(at 177.75425 178.9677)
+		(at 171.36 183.86)
 		(tags "P120PK-Y25BR10K ")
 		(property "Reference" "R79"
@@
 			(layers "*.Cu" "*.Mask")
 			(remove_unused_layers no)
-			(net "unconnected-(R79-Pad2)")
+			(net "Net-(U2A-PA7)")
 			(pinfunction "2_2")
 			(pintype "power_out")
@@
 			(layers "*.Cu" "*.Mask")
 			(remove_unused_layers no)
-			(net "Net-(R66-Pad2)")
+			(net "Net-(U2A-PC5)")
 			(pintype "passive")
 		)
@@
 		(layer "F.SilkS")
 	)
-	(gr_arc
-		(start 214.326764 337.990435)
-		(mid 113.735931 249.804834)
-		(end 187.999601 138.538835)
+	(gr_line
+		(start 187.999601 138.538835)
+		(end 395.295862 82.820341)
 		(stroke
-			(width 0.047065)
+			(width 0.05)
 			(type default)
 		)
 		(layer "Edge.Cuts")
 	)
-	(gr_line
-		(start 395.295862 82.821164)
-		(end 188.004137 138.538835)
+	(gr_arc
+		(start 214.326764 337.990435)
+		(mid 113.735931 249.804834)
+		(end 187.999601 138.538835)
 		(stroke
 			(width 0.047065)
@@
 	)
 	(gr_line
-		(start 395.295862 337.839872)
-		(end 214.323063 337.990478)
+		(start 214.326764 337.990435)
+		(end 395.295862 337.839872)
 		(stroke
-			(width 0.047065)
+			(width 0.05)
 			(type default)
 		)
@@
 	)
 	(via
-		(at 284.1 217.01)
-		(size 0.6)
-		(drill 0.3)
-		(layers "F.Cu" "B.Cu")
-		(free yes)
-		(net "GND")
-	)
-	(via
 		(at 286.12 233.34)
 		(size 0.6)
@@
 	)
 	(segment
+		(start 213.38 192.2)
+		(end 214.56 192.2)
+		(width 0.5)
+		(layer "F.Cu")
+		(net "Net-(U2A-PC5)")
+	)
+	(segment
+		(start 210.16 195.42)
+		(end 213.38 192.2)
+		(width 0.5)
+		(layer "F.Cu")
+		(net "Net-(U2A-PC5)")
+	)
+	(segment
+		(start 207.34 192.2)
+		(end 213.38 192.2)
+		(width 0.5)
+		(layer "F.Cu")
+		(net "Net-(U2A-PC5)")
+	)
+	(segment
+		(start 213.5 232.98)
+		(end 213.53 232.95)
+		(width 0.5)
+		(layer "F.Cu")
+		(net "Net-(U2A-PB1)")
+	)
+	(segment
+		(start 203.93 232.98)
+		(end 207.16 232.98)
+		(width 0.5)
+		(layer "F.Cu")
+		(net "Net-(U2A-PB1)")
+	)
+	(segment
+		(start 203.93 229.75)
+		(end 207.16 232.98)
+		(width 0.5)
+		(layer "F.Cu")
+		(net "Net-(U2A-PB1)")
+	)
+	(segment
+		(start 207.16 232.98)
+		(end 213.5 232.98)
+		(width 0.5)
+		(layer "F.Cu")
+		(net "Net-(U2A-PB1)")
+	)
+	(segment
 		(start 286.3381 230.450001)
 		(end 285.396101 230.450001)
@@
 	)
 	(segment
-		(start 213.5 232.98)
-		(end 213.53 232.95)
-		(width 0.5)
-		(layer "F.Cu")
-		(net "Net-(R52-Pad2)")
-	)
-	(segment
-		(start 203.93 232.98)
-		(end 207.16 232.98)
-		(width 0.5)
-		(layer "F.Cu")
-		(net "Net-(R52-Pad2)")
-	)
-	(segment
-		(start 203.93 229.75)
-		(end 207.16 232.98)
-		(width 0.5)
-		(layer "F.Cu")
-		(net "Net-(R52-Pad2)")
-	)
-	(segment
-		(start 207.16 232.98)
-		(end 213.5 232.98)
-		(width 0.5)
-		(layer "F.Cu")
-		(net "Net-(R52-Pad2)")
-	)
-	(segment
 		(start 189.790209 289.518886)
 		(end 189.790209 284.525209)
@@
 	)
 	(segment
-		(start 213.38 192.2)
-		(end 214.56 192.2)
-		(width 0.5)
-		(layer "F.Cu")
-		(net "Net-(R66-Pad2)")
-	)
-	(segment
-		(start 210.16 195.42)
-		(end 213.38 192.2)
-		(width 0.5)
-		(layer "F.Cu")
-		(net "Net-(R66-Pad2)")
-	)
-	(segment
-		(start 207.34 192.2)
-		(end 213.38 192.2)
-		(width 0.5)
-		(layer "F.Cu")
-		(net "Net-(R66-Pad2)")
-	)
-	(segment

Commit message: Power is pretty much fully routed, some data lines need to be routed. Final component locations established and confirmed by Jeremy and Ever.
Parts:
- moved R79 48.6 mm to (130.4, 210.0)
- moved R51 22.2 mm to (202.8, 204.4)
- moved R53 22.2 mm to (188.6, 204.4)
- moved R55 22.2 mm to (174.3, 204.4)
- moved R57 22.2 mm to (160.1, 204.4)
- moved R59 22.2 mm to (145.8, 204.4)
- moved S37 22.2 mm to (206.1, 199.4)
- moved S38 22.2 mm to (191.8, 199.4)
- moved S39 22.2 mm to (177.6, 199.4)
- moved S40 22.2 mm to (163.3, 199.4)
- moved S41 22.2 mm to (149.1, 199.4)
- moved U4 22.2 mm to (217.3, 196.9)
- moved R52 22.2 mm to (214.2, 207.6)
- moved R54 22.2 mm to (200.0, 207.6)
- moved R56 22.2 mm to (185.7, 207.6)
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Routing:
- net +3.3V: track 420.6 -> 612.9 mm
- net /DAC_schematic/DAC3: track 23.1 -> 58.9 mm
- net Net-(U1-1OUT): track 44.6 -> 79.8 mm
- net /DAC_schematic/DAC4: track 24.6 -> 58.9 mm
- net /DAC_schematic/DAC2: track 32.2 -> 59.0 mm
- net /DAC_schematic/DAC5: track 33.6 -> 59.0 mm
- net Net-(U1-2IN+): track 4.85 -> 24.4 mm, vias 0 -> 2
- net /DAC_schematic/DAC1: track 45.4 -> 59.0 mm
- net /DAC_schematic/DAC6: track 45.4 -> 59.0 mm
- net Net-(U2A-PH1-OSC_OUT): track 13.8 -> 22.6 mm
- net /DAC_schematic/DAC0: track 54.6 -> 59.1 mm
- net Net-(U2A-PH0-OSC_IN): track 15.8 -> 16.7 mm
- net GND: vias 42 -> 43

Commit message: PCB Revision 1.0 complete, Ground zones are filled, all components are wired, and holes are made for standoffs for case installment. Final changes to the onshape will need to be made to accomodate the pcb design
Connections:
- J3 pad 2: unconnected-(J3-Pad2) -> GND
- R52 pad 2: Net-(U2A-PB1) -> Net-(U2A-PB0)
- R64 pad 2: Net-(U2A-PB1) -> Net-(U2A-PB0)
- R66 pad 2: Net-(U2A-PC5) -> Net-(U2A-PA7)
- R67 pad 1: Net-(U2A-PC5) -> Net-(U2A-PA7)
- R79 pad 2: Net-(U2A-PA7) -> Net-(U2A-PB1)
- U4 pad 4: Net-(U2A-PB0) -> Net-(U2A-PC5)
Routing:
- net Net-(U2A-PB1): track 14.2 -> 156.5 mm
- net Net-(U2A-PA7): track 0.00 -> 103.5 mm
- net Net-(U2A-PB0): track 0.00 -> 91.2 mm
- net Net-(U2A-PC4): track 0.00 -> 76.6 mm
- net Net-(U2A-PC5): track 11.8 -> 71.6 mm
- net +3.3V: track 612.9 -> 620.6 mm, vias 18 -> 19
- net GND: vias 43 -> 1524
- added copper zone on B.Cu, net GND
- added copper zone on F.Cu, net GND
Other:
- outline, holes or cut-outs redrawn
- board text added: "BAT 1 PWR | GND"
- board text added: "BAT 2 PWR | GND"
- board text added: "BAT 3 PWR | GND"
- board text added: "SHLD / GND"
- board text removed: "BAT 1 PWR / GND"
- board text removed: "BAT 2 PWR / GND"
- board text removed: "BAT 3 PWR / GND"
- board text removed: "SLD / GND"
