File: synthia/synthia.kicad_pcb (KiCad board)
At the start: 2 copper layers, 282.4 x 255.2 mm, 229 parts, among them J1 MJ-63022B, J2 SJ3-35083C-TR, J3 PJ-007, J4 SDS-50J, Q1 IRF9540N, U1 TLV272IP, U2 STM32H750ZBT6, U3 LD1117V33, U4 PVA1EEH31.2NV2, U5 PVA1EEH31.2NV2, U6 ATS08A-E

Commit message: Made slight efficiency improvements to wiring.
Routing:
- net Net-(U1-1OUT): track 79.8 -> 79.1 mm
- net Net-(U1-2IN-): track 53.2 -> 52.6 mm
Changed lines of the file:
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@@
-	)
-	(segment
-		(start 333.71 123.64)
-		(end 344.29 123.64)
-		(width 0.6)
-		(layer "F.Cu")
-		(net "Net-(U1-1OUT)")
 	)
 	(segment
@@
 	(segment
 		(start 342.56 98.78)
-		(end 354.91 98.78)
+		(end 353.43 98.78)
 		(width 0.6)
 		(layer "F.Cu")
@@
 	)
 	(segment
+		(start 354.86 100.21)
+		(end 354.86 100.98)
+		(width 0.6)
+		(layer "F.Cu")
+		(net "Net-(U1-1OUT)")
+	)
+	(segment
 		(start 333.71 125.54)
 		(end 333.71 123.64)
@@
 	)
 	(segment
+		(start 334.21 123.64)
+		(end 344.29 123.64)
+		(width 0.6)
+		(layer "F.Cu")
+		(net "Net-(U1-1OUT)")
+	)
+	(segment
 		(start 360.33 129.49)
 		(end 362.83425 126.98575)
@@
 	)
 	(segment
-		(start 354.91 98.78)
-		(end 354.91 100.93)
+		(start 333.71 123.14)
+		(end 333.71 123.64)
+		(width 0.6)
+		(layer "F.Cu")
+		(net "Net-(U1-1OUT)")
+	)
+	(segment
+		(start 353.43 98.78)
+		(end 354.86 100.21)
 		(width 0.6)
 		(layer "F.Cu")
@@
 	(segment
 		(start 333.71 122.35)
-		(end 333.71 123.64)
+		(end 333.71 123.14)
+		(width 0.6)
+		(layer "F.Cu")
+		(net "Net-(U1-1OUT)")
+	)
+	(segment
+		(start 333.71 123.14)
+		(end 334.21 123.64)
 		(width 0.6)
 		(layer "F.Cu")
@@
 	(segment
 		(start 343.24 130.62)
-		(end 345.16 130.62)
+		(end 344.19 130.62)
 		(width 0.8)
 		(layer "F.Cu")
@@
 	)
 	(segment
-		(start 343.24 130.16)
-		(end 343.24 130.62)
-		(width 0.8)
-		(layer "F.Cu")
-		(net "Net-(U1-2IN-)")
-	)
-	(segment
-		(start 343.23 130.17)
-		(end 343.24 130.16)
-		(width 0.5)
-		(layer "F.Cu")
-		(net "Net-(U1-2IN-)")
-	)
-	(segment
-		(start 343.24 130.16)
-		(end 343.24 128.08)
+		(start 344.19 130.62)
+		(end 345.16 130.62)
 		(width 0.8)
 		(layer "F.Cu")
@@
 	)
 	(segment
-		(start 343.24 128.08)
-		(end 341.65 128.08)
-		(width 0.8)
-		(layer "F.Cu")
+		(start 341.65 128.08)
+		(end 344.19 130.62)
+		(width 0.8)
+		(layer "F.Cu")
